File: Projekt/Projekt.kicad_sch (KiCad schematic)
At the start: 5 parts, among them U1 STM32G071KxT

Commit message: Add files via upload
Parts:
- removed R?, czujnik_opadów: R, symbol Device:R
- removed U?: LM358, symbol Amplifier_Operational:LM358
- removed U?: LCD-016N002L, Display:LCD-016N002L, symbol Display_Character:LCD-016N002L
- added C? (x3): 100nF, symbol Device:C_Small
- added J2: Valve output ground, symbol Connector:Conn_01x04_Male
- added J3: Valve input +24V, symbol Connector:Conn_01x04_Male
- added J?: Conn_01x06, Connector_PinHeader_1.00mm:PinHeader_1x06_P1.00mm_Vertical_SMD_Pin1Left, symbol Connector_Generic:Conn_01x06
- added Q1: Valve 1 power, Package_DirectFET:DirectFET_MD, symbol Transistor_FET:IRL6283M
- added Q2: Valve 2 power, Package_DirectFET:DirectFET_MD, symbol Transistor_FET:IRL6283M
- added Q3: Valve 3 power, Package_DirectFET:DirectFET_MD, symbol Transistor_FET:IRL6283M
- added Q4: Valve 4 power, Package_DirectFET:DirectFET_MD, symbol Transistor_FET:IRL6283M
- added R?: 100k, symbol Device:R_Small
- added RV?: R_Potentiometer_Small, symbol Device:R_Potentiometer_Small
- added U?: NHD-0420H1Z, Display:NHD-0420H1Z, symbol Display_Character:NHD-0420H1Z
Connections:
- net GND: now also C?.2, C?.2, C?.2, J2.1 (Pin_1), J2.2 (Pin_2), J2.3 (Pin_3), J2.4 (Pin_4), J?.3 (Pin_3), RV?.3, U?.1 (VSS)
- net at U1.6 (~{RST}/PF2): now also R?.1
- net +5V renamed +3.3V
- net +3.3V: now also C?.1, C?.1, C?.1, J?.1 (Pin_1), R?.2, RV?.1, U?.2 (VDD)
- new net: RV?.2, U?.3 (VO)
- new net +24V: Q1.3 (S), Q2.3 (S), Q3.3 (S), Q4.3 (S)
- new net NRST: J?.5 (Pin_5)
- new net Q1: Q1.2 (G)
- new net Q2: Q2.2 (G)
- new net Q3: Q3.2 (G)
- new net Q4: Q4.2 (G)
- new net SWCLK: J?.2 (Pin_2)
- new net SWDIO: J?.4 (Pin_4)
- new net V1: J3.1 (Pin_1), Q1.1 (D)
- new net V2: J3.2 (Pin_2), Q2.1 (D)
- new net V3: J3.3 (Pin_3), Q3.1 (D)
- new net V4: J3.4 (Pin_4), Q4.1 (D)
- no-connect marks 0 -> 1
Other:
- added sheet Power supply (power_supply.kicad_sch)
- added sheet Sensors (sensors.kicad_sch)
- added sheet buttons (buttons.kicad_sch)
- note added: "5V"
- note added: "GND"
- note added: "NRST"
- note added: "SWCLK"
- note added: "SWDIO"
- note added: "SWO"
- note added: "VDD"
- note added: "Valve"
- note added: "filtr dolnoprzepustowy"
- note added: "złącze programatora ()"
- moved on the sheet: U1

Commit message: Add files via upload
Parts:
- added R?: 100k, symbol Device:R
- added R? (x2): 10k, symbol Device:R
- added U3: ESP-12E, RF_Module:ESP-12E, symbol RF_Module:ESP-12E
- added U6: DS1307N+, Package_DIP:DIP-8_W7.62mm, symbol Timer_RTC:DS1307N+
- gave numbers to parts that had none: 1
Connections:
- net +3.3V: now also R?.1, U3.8 (VCC)
- net GND: now also U3.15 (GND), U6.4 (GND)
- new net: R?.2, U3.1 (~{RST})
- new net: R?.2, U6.5 (SDA)
- new net: R?.2, U6.6 (SCL)
- new net +5V: R?.1, R?.1, U6.8 (VCC)
Other:
- note added: "to powinno iść jeszcze na piny ale nie wiemy jeszcze jakie"
- moved on the sheet: RV?, U2

Commit message: Add files via upload
Parts:
- removed C? (x3): 100nF, symbol Device:C_Small
- removed R? (x2): 10k, symbol Device:R
- removed RV?: R_Potentiometer_Small, symbol Device:R_Potentiometer_Small
- added R1, R2, R3, R4: 10k, symbol Device:R
- added U3: PCF8574, symbol Interface_Expansion:PCF8574
- gave numbers to parts that had none: 3
- renumbered J3 to J1, Q3 to Q2, Q2 to Q3, U6 to U1, U1 to U2, U2 to U4, U3 to U5
Connections:
- net +3.3V: now also U3.16 (VDD); no longer U4.2 (VDD)
- net GND: now also U3.8 (VSS); no longer U4.1 (VSS)
- net Q1: now also U2.15 (PB0), R1.2; no longer Q1.2 (G)
- net Q2: now also U2.16 (PB1), R3.2; no longer Q3.2 (G)
- net Q3: now also U2.17 (PB2), R2.2; no longer Q2.2 (G)
- net Q4: now also U2.27 (PB3), R4.2; no longer Q4.2 (G)
- net SW1: now also U2.28 (PB4)
- net SW2: now also U2.29 (PB5)
- net SW3: now also U2.30 (PB6)
- net SW4: now also U2.31 (PB7)
- net SW5: now also U2.32 (PB8)
- net SW6: now also U2.1 (PB9)
- net I2C2_SDA: now reaches U1.5 (SDA)
- net I2C2_SDA: now also U2.23 (PA12_[PA10])
- net I2C2_SCL: now reaches U1.6 (SCL)
- net I2C2_SCL: now also U2.22 (PA11_[PA9])
- net ADC1_IN4: now reaches U5.2 (ADC)
- net ADC1_IN4: now also U2.11 (PA4)
- net I2C1_SCL: now reaches U2.19 (PA9)
- net I2C1_SCL: now also U3.14 (SCL)
- net GPIO_Input: now reaches U2.20 (PC6)
- net I2C1_SDA: now reaches U2.21 (PA10)
- net I2C1_SDA: now also U3.15 (SDA)
- net ADC_IN1: now reaches U2.8 (PA1)
- net at U4.10 (DB3): now also U3.7 (P3)
- net at U4.11 (DB4): now also U3.9 (P4)
- net at U4.12 (DB5): now also U3.10 (P5)
- net at U4.13 (DB6): now also U3.11 (P6)
- net at U4.14 (DB7): now also U3.12 (P7)
- net at U4.7 (DB0): now also U3.4 (P0)
- net at U4.8 (DB1): now also U3.5 (P1)
- net at U4.9 (DB2): now also U3.6 (P2)
- new net: Q4.2 (G), R4.1
- new net: Q3.2 (G), R3.1
- new net: Q1.2 (G), R1.1
- new net: Q2.2 (G), R2.1
Other:
- sheet buttons renamed Buttons
- note added: "LCD 4x20 with connector"
- note added: "Real Time Clock"
- note removed: "5V"
- note removed: "filtr dolnoprzepustowy"
- note removed: "to powinno iść jeszcze na piny ale nie wiemy jeszcze jakie"
- moved on the sheet: J1, J2, J3, Q1, Q2, Q3, Q4, R5, R6, U1, U2, U4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

Commit message: Add files via upload
Parts:
- removed R5: 100k, symbol Device:R_Small
- added BT1, BT2: 3V, Battery:BatteryHolder_Keystone_500, symbol Device:Battery_Cell
- added C1, C2: 12.5pF, Capacitor_SMD:C_0603_1608Metric, symbol Device:C
- added C3, C4, C5, C6, C7, C8: 100nF, Capacitor_SMD:C_0603_1608Metric, symbol Device:C
- added R1, R2: 3k, Resistor_SMD:R_0603_1608Metric, symbol Device:R
- added Y1: 32.768KHZ, Crystal:Crystal_SMD_FOX_FQ7050-2Pin_7.0x5.0mm, symbol Device:Crystal
- J1, J2: footprint (none) -> Connector_Wire:SolderWire-0.1sqmm_1x04_P3.6mm_D0.4mm_OD1mm
- R3: renamed from R1; footprint (none) -> Resistor_SMD:R_0603_1608Metric
- R4: renamed from R2; footprint (none) -> Resistor_SMD:R_0603_1608Metric
- R5: renamed from R3; footprint (none) -> Resistor_SMD:R_0603_1608Metric
- R6: renamed from R4; footprint (none) -> Resistor_SMD:R_0603_1608Metric
- R7: renamed from R6; footprint (none) -> Resistor_SMD:R_0603_1608Metric
- U3: footprint (none) -> Package_DIP:DIP-16_W7.62mm
Connections:
- net +3.3V: now also R7.2, U4.2 (VDD), U5.1 (~{RST}), C5.1, C6.1, C7.1, C8.1
- net +5V: now also C3.1, C4.1, R1.1, R2.1
- net GND: now also U4.1 (VSS), BT1.2 (-), C1.2, C2.2, C3.2, C4.2, C5.2, C6.2, C7.2, C8.2
- net I2C2_SCL: now also R1.2, R2.2
- net NRST: now also U2.6 (~{RST}/PF2)
- net SWCLK: now also U2.25 (PA14/BOOT0)
- net SWDIO: now also U2.24 (PA13)
- net at U1.1 (X1): now also C1.1, Y1.2
- net at U1.2 (X2): now also C2.1, Y1.1
- net at U1.3 (VBAT): now also BT1.1 (+)
- net USART2_RX: now reaches U5.21 (GPIO3/RXD)
- net USART2_RX: now also U2.10 (PA3)
- net USART2_TX: now reaches U5.22 (GPIO1/TXD)
- net USART2_TX: now also U2.9 (PA2)
- net at U4.15 (A): now also BT2.1 (+)
- net at U4.16 (K): now also BT2.2 (-)
- net GPIO_Input renamed Dout
- no-connect marks 1 -> 32
Other:
- note added: "WIFI_MODULE"
- moved on the sheet: J1, J2, J3, Q1, Q2, Q3, Q4, R3, R4, R5, R6, R7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
