File: Projekt/buttons.kicad_sch (KiCad schematic)
At the start: 6 parts, among them SW1 SW_MEC_5E, SW2 SW_MEC_5E, SW3 SW_MEC_5E, SW4 SW_MEC_5E, SW5 SW_MEC_5E, SW6 SW_MEC_5E

Commit message: Add files via upload
Parts:
- SW1, SW2, SW3, SW4, SW5, SW6: footprint (none) -> Button_Switch_SMD:SW_SPST_B3S-1000
Connections:
- no-connect marks 0 -> 12
Changed lines of the file:
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@@
 (kicad_sch (version 20211123) (generator eeschema)
   (paper "A4")
+  (no_connect (at 38.1 85.09))
+  (no_connect (at 48.26 82.55))
+  (no_connect (at 77.47 59.69))
+  (no_connect (at 87.63 57.15))
+  (no_connect (at 38.1 59.69))
+  (no_connect (at 48.26 57.15))
+  (no_connect (at 77.47 85.09))
+  (no_connect (at 87.63 82.55))
+  (no_connect (at 38.1 34.29))
+  (no_connect (at 48.26 31.75))
+  (no_connect (at 77.47 34.29))
+  (no_connect (at 87.63 31.75))
   (wire (pts (xy 52.07 86.36) (xy 52.07 85.09))
     (stroke (width 0) (type default) (color 0 0 0 0))
@@
     (property "Reference" "SW1" (id 0) (at 43.18 24.13 0))
     (property "Value" "SW_MEC_5E" (id 1) (at 43.18 26.67 0))
-    (property "Footprint" "" (id 2) (at 43.18 26.67 0)
+    (property "Footprint" "Button_Switch_SMD:SW_SPST_B3S-1000" (id 2) (at 43.18 26.67 0)
       (effects (font (size 1.27 1.27)) hide)
     )
@@
   (symbol (lib_id "power:GND") (at 52.07 60.96 0) (unit 1)
     (in_bom yes) (on_board yes) (fields_autoplaced)
-    (property "Reference" "#PWR021" (id 0) (at 52.07 67.31 0)
+    (property "Reference" "#PWR029" (id 0) (at 52.07 67.31 0)
       (effects (font (size 1.27 1.27)) hide)
     )
@@
   (symbol (lib_id "power:GND") (at 91.44 86.36 0) (unit 1)
     (in_bom yes) (on_board yes) (fields_autoplaced)
-    (property "Reference" "#PWR025" (id 0) (at 91.44 92.71 0)
+    (property "Reference" "#PWR033" (id 0) (at 91.44 92.71 0)
       (effects (font (size 1.27 1.27)) hide)
     )
@@
     (property "Reference" "SW2" (id 0) (at 43.18 49.53 0))
     (property "Value" "SW_MEC_5E" (id 1) (at 43.18 52.07 0))
-    (property "Footprint" "" (id 2) (at 43.18 52.07 0)
+    (property "Footprint" "Button_Switch_SMD:SW_SPST_B3S-1000" (id 2) (at 43.18 52.07 0)
       (effects (font (size 1.27 1.27)) hide)
     )
@@
   (symbol (lib_id "power:GND") (at 91.44 35.56 0) (unit 1)
     (in_bom yes) (on_board yes) (fields_autoplaced)
-    (property "Reference" "#PWR023" (id 0) (at 91.44 41.91 0)
+    (property "Reference" "#PWR031" (id 0) (at 91.44 41.91 0)
       (effects (font (size 1.27 1.27)) hide)
     )
@@
     (property "Reference" "SW5" (id 0) (at 82.55 49.53 0))
     (property "Value" "SW_MEC_5E" (id 1) (at 82.55 52.07 0))
-    (property "Footprint" "" (id 2) (at 82.55 52.07 0)
+    (property "Footprint" "Button_Switch_SMD:SW_SPST_B3S-1000" (id 2) (at 82.55 52.07 0)
       (effects (font (size 1.27 1.27)) hide)
     )
@@
     (property "Reference" "SW6" (id 0) (at 82.55 74.93 0))
     (property "Value" "SW_MEC_5E" (id 1) (at 82.55 77.47 0))
-    (property "Footprint" "" (id 2) (at 82.55 77.47 0)
+    (property "Footprint" "Button_Switch_SMD:SW_SPST_B3S-1000" (id 2) (at 82.55 77.47 0)
       (effects (font (size 1.27 1.27)) hide)
     )
@@
   (symbol (lib_id "power:GND") (at 52.07 86.36 0) (unit 1)
     (in_bom yes) (on_board yes) (fields_autoplaced)
-    (property "Reference" "#PWR022" (id 0) (at 52.07 92.71 0)
+    (property "Reference" "#PWR030" (id 0) (at 52.07 92.71 0)
       (effects (font (size 1.27 1.27)) hide)
     )
@@
   (symbol (lib_id "power:GND") (at 91.44 60.96 0) (unit 1)
     (in_bom yes) (on_board yes) (fields_autoplaced)
-    (property "Reference" "#PWR024" (id 0) (at 91.44 67.31 0)
+    (property "Reference" "#PWR032" (id 0) (at 91.44 67.31 0)
       (effects (font (size 1.27 1.27)) hide)
     )
@@
   (symbol (lib_id "power:GND") (at 52.07 35.56 0) (unit 1)
     (in_bom yes) (on_board yes) (fields_autoplaced)
-    (property "Reference" "#PWR020" (id 0) (at 52.07 41.91 0)
+    (property "Reference" "#PWR028" (id 0) (at 52.07 41.91 0)
       (effects (font (size 1.27 1.27)) hide)
     )
@@
     (property "Reference" "SW4" (id 0) (at 82.55 24.13 0))
     (property "Value" "SW_MEC_5E" (id 1) (at 82.55 26.67 0))
-    (property "Footprint" "" (id 2) (at 82.55 26.67 0)
+    (property "Footprint" "Button_Switch_SMD:SW_SPST_B3S-1000" (id 2) (at 82.55 26.67 0)
       (effects (font (size 1.27 1.27)) hide)
     )
@@
     (property "Reference" "SW3" (id 0) (at 43.18 74.93 0))
     (property "Value" "SW_MEC_5E" (id 1) (at 43.18 77.47 0))
-    (property "Footprint" "" (id 2) (at 43.18 77.47 0)
-      (effects (font (size 1.27 1.27)) hide)
-    )
+    (property "Footprint" "Button_Switch_SMD:SW_SPST_B3S-1000" (id 2) (at 43.18 77.47 0)
+      (effects (font (size 1.27 1.27)) hide)
+    )
