File: Projekt/power_supply.kicad_sch (KiCad schematic)
At the start: 14 parts

Commit message: Add files via upload
Parts:
- gave numbers to parts that had none: 2
Changed lines of the file:
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@@
   (symbol (lib_id "Regulator_Linear:LM1117-3.3") (at 186.69 44.45 0) (unit 1)
     (in_bom yes) (on_board yes)
-    (property "Reference" "U?" (id 0) (at 186.69 38.1 0))
+    (property "Reference" "U5" (id 0) (at 186.69 38.1 0))
     (property "Value" "LM1117-3.3" (id 1) (at 186.69 40.64 0))
     (property "Footprint" "Package_TO_SOT_SMD:SOT-223-3_TabPin2" (id 2) (at 186.69 44.45 0)
@@
   (symbol (lib_id "Regulator_Switching:AOZ1280CI") (at 104.14 44.45 0) (unit 1)
     (in_bom yes) (on_board yes)
-    (property "Reference" "U?" (id 0) (at 104.14 35.56 0))
+    (property "Reference" "U4" (id 0) (at 104.14 35.56 0))
     (property "Value" "AOZ1280CI" (id 1) (at 104.14 38.1 0))
     (property "Footprint" "Package_TO_SOT_SMD:SOT-23-6" (id 2) (at 121.92 50.8 0)

Commit message: Add files via upload
Parts:
- removed C?: 10μF, Capacitor_SMD:C_Elec_4x5.4, symbol Device:C_Polarized_Small
- removed C? (x3): 100nF, Capacitor_SMD:C_0603_1608Metric, symbol Device:C_Small
- removed C?: 10nF, Capacitor_SMD:C_0603_1608Metric, symbol Device:C_Small
- removed C?: 4.7μF, Capacitor_SMD:C_Elec_4x5.4, symbol Device:C_Polarized_Small
- removed D?: SK32SMA, Diode_SMD:D_SMA, symbol Device:D_Schottky_Small
- removed F?: 500mA, Fuse:Fuse_1210_3225Metric, symbol Device:Polyfuse_Small
- removed L?: 2.2μH, Inductor_SMD:L_Bourns-SRN4018, symbol Device:L_Small
- removed R?: 10kΩ, Resistor_SMD:R_0603_1608Metric, symbol Device:R_Small
- removed R?: 4.7kΩ, Resistor_SMD:R_0603_1608Metric, symbol Device:R_Small
- removed R?: 33kΩ, Resistor_SMD:R_0603_1608Metric, symbol Device:R_Small
- removed U4: AOZ1280CI, Package_TO_SOT_SMD:SOT-23-6, symbol Regulator_Switching:AOZ1280CI
- removed U5: LM1117-3.3, Package_TO_SOT_SMD:SOT-223-3_TabPin2, symbol Regulator_Linear:LM1117-3.3
- added C3: 2.2uF, symbol Device:C
- added L1: 18uH, symbol Device:L
- added PS1: IA0503S, Converter_DCDC:Converter_DCDC_XP_POWER-IAxxxxS_THT, symbol Converter_DCDC:IA0503S
- added U7: ATA00A18S-L, Converter_DCDC:Converter_DCDC_Artesyn_ATA_SMD, symbol Converter_DCDC:ATA00A18S-L
Connections:
- net GND: now also PS1.4 (-Vout), U7.1 (-VIN)
- new net: C3.2, PS1.2 (-Vin), U7.10 (-VOUT)
- new net: L1.2, PS1.1 (+Vin)
- new net +24V: U7.16 (+VIN)
- new net 3.3V Output: PS1.6 (+Vout)
- new net 5V Output: C3.1, L1.1, U7.9 (+VOUT)
Other:
- note removed: "Buck converter output voltage: Vout = Vref * (1 + R5 / R6) Vout = 0.8 * (1 + 33k / 4.7k) = 6.42 V"

Commit message: Add files via upload
Parts:
- C11: renamed from C3; footprint (none) -> Capacitor_SMD:C_0603_1608Metric
- L1: footprint (none) -> Inductor_SMD:L_0603_1608Metric
Connections:
- no-connect marks 0 -> 2
Changed lines of the file:
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@@
   (junction (at 134.62 46.99) (diameter 0) (color 0 0 0 0)
   )
+  (no_connect (at 100.33 44.45))
+  (no_connect (at 176.53 41.91))
   (wire (pts (xy 125.73 46.99) (xy 125.73 44.45))
     (stroke (width 0) (type default) (color 0 0 0 0))
@@
   (symbol (lib_id "Device:C") (at 134.62 43.18 0) (unit 1)
     (in_bom yes) (on_board yes) (fields_autoplaced)
-    (property "Reference" "C3" (id 0) (at 138.235 41.9099 0)
+    (property "Reference" "C11" (id 0) (at 138.235 41.9099 0)
       (effects (font (size 1.27 1.27)) (justify left))
     )
@@
       (effects (font (size 1.27 1.27)) (justify left))
     )
-    (property "Footprint" "" (id 2) (at 135.5852 46.99 0)
+    (property "Footprint" "Capacitor_SMD:C_0603_1608Metric" (id 2) (at 135.5852 46.99 0)
       (effects (font (size 1.27 1.27)) hide)
     )
@@
   (symbol (lib_id "power:+24V") (at 96.52 39.37 0) (unit 1)
     (in_bom yes) (on_board yes) (fields_autoplaced)
-    (property "Reference" "#PWR027" (id 0) (at 96.52 43.18 0)
+    (property "Reference" "#PWR035" (id 0) (at 96.52 43.18 0)
       (effects (font (size 1.27 1.27)) hide)
     )
@@
     (property "Reference" "L1" (id 0) (at 146.05 33.02 90))
     (property "Value" "18uH" (id 1) (at 146.05 35.56 90))
-    (property "Footprint" "" (id 2) (at 146.05 39.37 0)
+    (property "Footprint" "Inductor_SMD:L_0603_1608Metric" (id 2) (at 146.05 39.37 0)
       (effects (font (size 1.27 1.27)) hide)
     )
@@
   (symbol (lib_id "power:GND") (at 95.25 49.53 0) (unit 1)
     (in_bom yes) (on_board yes) (fields_autoplaced)
-    (property "Reference" "#PWR026" (id 0) (at 95.25 55.88 0)
+    (property "Reference" "#PWR034" (id 0) (at 95.25 55.88 0)
       (effects (font (size 1.27 1.27)) hide)
     )
@@
   (symbol (lib_id "power:GND") (at 179.07 48.26 0) (unit 1)
     (in_bom yes) (on_board yes) (fields_autoplaced)
-    (property "Reference" "#PWR028" (id 0) (at 179.07 54.61 0)
+    (property "Reference" "#PWR036" (id 0) (at 179.07 54.61 0)
       (effects (font (size 1.27 1.27)) hide)
     )
