File: Projekt/sensors.kicad_sch (KiCad schematic)
At the start: 11 parts, among them J1 Conn_01x02, U1 LM393

Commit message: Add files via upload
Parts:
- removed C? (x2): C, symbol Device:C
- removed D? (x2): LED, symbol Device:LED
- removed J1: Conn_01x02, symbol Connector_Generic:Conn_01x02
- removed R5, R? (x2): R, symbol Device:R
- removed RV?: R_Potentiometer, symbol Device:R_Potentiometer
- removed U1, U?: LM393, symbol Comparator:LM393
- added C1, C2: 104, symbol Device:C
- added D1: Trigger LED, symbol Device:LED
- added D2: Power LED, symbol Device:LED
- added J4: Conn_01x02, symbol Connector_Generic:Conn_01x02
- added R7: 10k, symbol Device:R
- added R8, R9: 1k, symbol Device:R
- added RV1: 10k, symbol Device:R_Potentiometer
- added U6: LM393, symbol Comparator:LM393
Connections:
- net Aout: now also C1.1, J4.2 (Pin_2), R7.2, U6.3 (+)
- net Dout: now also R8.2, U6.1
- net GND: now also C1.2, C2.2, D2.1 (K), J4.1 (Pin_1), RV1.3, U6.4 (V-)
- net VCC: now also D1.2 (A), R7.1, R9.1, RV1.1, U6.8 (V+)
- new net: D1.1 (K), R8.1
- new net: C2.1, RV1.2, U6.2 (-)
- new net: D2.2 (A), R9.2
Other:
- note added: "Soil Moisture Sensor Input"
- note removed: "Soil dampness sensor"

Commit message: Add files via upload
Parts:
- C10: renamed from C2; footprint (none) -> Capacitor_SMD:C_0603_1608Metric
- C9: renamed from C1; footprint (none) -> Capacitor_SMD:C_0603_1608Metric
- D1, D2: footprint (none) -> LED_SMD:LED_0603_1608Metric
- J4: footprint (none) -> Connector_Wire:SolderWire-0.1sqmm_1x02_P3.6mm_D0.4mm_OD1mm
- R10: renamed from R9; footprint (none) -> Resistor_SMD:R_0603_1608Metric
- R8: renamed from R7; footprint (none) -> Resistor_SMD:R_0603_1608Metric
- R9: renamed from R8; footprint (none) -> Resistor_SMD:R_0603_1608Metric
- RV1: footprint (none) -> Potentiometer_SMD:Potentiometer_ACP_CA6-VSMD_Vertical
- U6: footprint (none) -> Package_DIP:DIP-8_W7.62mm_Socket
Changed lines of the file:
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@@
   (symbol (lib_id "Device:R") (at 111.76 43.18 0) (unit 1)
     (in_bom yes) (on_board yes) (fields_autoplaced)
-    (property "Reference" "R8" (id 0) (at 114.3 41.9099 0)
+    (property "Reference" "R9" (id 0) (at 114.3 41.9099 0)
       (effects (font (size 1.27 1.27)) (justify left))
     )
@@
       (effects (font (size 1.27 1.27)) (justify left))
     )
-    (property "Footprint" "" (id 2) (at 109.982 43.18 90)
+    (property "Footprint" "Resistor_SMD:R_0603_1608Metric" (id 2) (at 109.982 43.18 90)
       (effects (font (size 1.27 1.27)) hide)
     )
@@
     (property "Reference" "J4" (id 0) (at 30.48 43.18 0))
     (property "Value" "Conn_01x02" (id 1) (at 30.48 45.72 0))
-    (property "Footprint" "" (id 2) (at 30.48 52.07 0)
+    (property "Footprint" "Connector_Wire:SolderWire-0.1sqmm_1x02_P3.6mm_D0.4mm_OD1mm" (id 2) (at 30.48 52.07 0)
       (effects (font (size 1.27 1.27)) hide)
     )
@@
       (effects (font (size 1.27 1.27)) (justify right))
     )
-    (property "Footprint" "" (id 2) (at 66.04 62.23 0)
+    (property "Footprint" "Potentiometer_SMD:Potentiometer_ACP_CA6-VSMD_Vertical" (id 2) (at 66.04 62.23 0)
       (effects (font (size 1.27 1.27)) hide)
     )
@@
   (symbol (lib_id "Device:C") (at 52.07 62.23 0) (unit 1)
     (in_bom yes) (on_board yes) (fields_autoplaced)
-    (property "Reference" "C1" (id 0) (at 55.88 60.9599 0)
+    (property "Reference" "C9" (id 0) (at 55.88 60.9599 0)
       (effects (font (size 1.27 1.27)) (justify left))
     )
@@
       (effects (font (size 1.27 1.27)) (justify left))
     )
-    (property "Footprint" "" (id 2) (at 53.0352 66.04 0)
+    (property "Footprint" "Capacitor_SMD:C_0603_1608Metric" (id 2) (at 53.0352 66.04 0)
       (effects (font (size 1.27 1.27)) hide)
     )
@@
   (symbol (lib_id "Device:R") (at 120.65 39.37 0) (unit 1)
     (in_bom yes) (on_board yes) (fields_autoplaced)
-    (property "Reference" "R9" (id 0) (at 123.19 38.0999 0)
+    (property "Reference" "R10" (id 0) (at 123.19 38.0999 0)
       (effects (font (size 1.27 1.27)) (justify left))
     )
@@
       (effects (font (size 1.27 1.27)) (justify left))
     )
-    (property "Footprint" "" (id 2) (at 118.872 39.37 90)
+    (property "Footprint" "Resistor_SMD:R_0603_1608Metric" (id 2) (at 118.872 39.37 90)
       (effects (font (size 1.27 1.27)) hide)
     )
@@
   (symbol (lib_id "Device:R") (at 40.64 36.83 0) (unit 1)
     (in_bom yes) (on_board yes) (fields_autoplaced)
-    (property "Reference" "R7" (id 0) (at 43.18 35.5599 0)
+    (property "Reference" "R8" (id 0) (at 43.18 35.5599 0)
       (effects (font (size 1.27 1.27)) (justify left))
     )
@@
       (effects (font (size 1.27 1.27)) (justify left))
     )
-    (property "Footprint" "" (id 2) (at 38.862 36.83 90)
+    (property "Footprint" "Resistor_SMD:R_0603_1608Metric" (id 2) (at 38.862 36.83 90)
       (effects (font (size 1.27 1.27)) hide)
     )
@@
     (property "Reference" "U6" (id 0) (at 99.06 44.45 0))
     (property "Value" "LM393" (id 1) (at 100.33 46.99 0))
-    (property "Footprint" "" (id 2) (at 95.25 52.07 0)
+    (property "Footprint" "Package_DIP:DIP-8_W7.62mm_Socket" (id 2) (at 95.25 52.07 0)
       (effects (font (size 1.27 1.27)) hide)
     )
@@
       (effects (font (size 1.27 1.27)) (justify right))
     )
-    (property "Footprint" "" (id 2) (at 120.65 60.96 0)
+    (property "Footprint" "LED_SMD:LED_0603_1608Metric" (id 2) (at 120.65 60.96 0)
       (effects (font (size 1.27 1.27)) hide)
     )
@@
       (effects (font (size 1.27 1.27)) (justify right))
     )
-    (property "Footprint" "" (id 2) (at 111.76 31.75 0)
+    (property "Footprint" "LED_SMD:LED_0603_1608Metric" (id 2) (at 111.76 31.75 0)
       (effects (font (size 1.27 1.27)) hide)
     )
@@
       (effects (font (size 1.27 1.27)) (justify left))
     )
-    (property "Footprint" "" (id 2) (at 97.79 52.07 0)
+    (property "Footprint" "Package_DIP:DIP-8_W7.62mm_Socket" (id 2) (at 97.79 52.07 0)
       (effects (font (size 1.27 1.27)) hide)
     )
@@
   (symbol (lib_id "Device:C") (at 76.2 62.23 0) (unit 1)
     (in_bom yes) (on_board yes) (fields_autoplaced)
-    (property "Reference" "C2" (id 0) (at 80.01 60.9599 0)
+    (property "Reference" "C10" (id 0) (at 80.01 60.9599 0)
       (effects (font (size 1.27 1.27)) (justify left))
     )
@@
       (effects (font (size 1.27 1.27)) (justify left))
     )
-    (property "Footprint" "" (id 2) (at 77.1652 66.04 0)
+    (property "Footprint" "Capacitor_SMD:C_0603_1608Metric" (id 2) (at 77.1652 66.04 0)
       (effects (font (size 1.27 1.27)) hide)
     )
